Commit message: PID gains updated. ft_tool xacro model meged with new frames for local depth camera

File: kuka_control/models/camera/kinect_camera.urdf.xacro (robot description, xacro)
@@ -64,5 +64,5 @@
             <horizontal_fov>${60 * M_PI/180.0}</horizontal_fov>
             <image>
-              <format>B8G8R8</format>-->
+              <format>R8G8B8</format>
               <!--<width>640</width>
               <height>480</height>-->

File: kuka_control/models/ft_tool.xacro (robot description, xacro)
@@ -24,5 +24,6 @@
   <xacro:include filename="$(find kuka_control)/models/realsense/realsense_d435.xacro" />
   <xacro:realsense parent="brida_link" name="camera">
-      <origin xyz="0.0739 -0.0306 0.01" rpy="0 ${-M_PI/2} ${M_PI-M_PI/8}" />
+   <!--   <origin xyz="0.0739 -0.0306 0.01" rpy="0 ${-M_PI/2} ${M_PI-M_PI/8}" />-->
+	<origin xyz="0.13 0.05 0.025" rpy="${-2.0*M_PI/180} ${-M_PI/2+30.0*M_PI/180} ${M_PI+M_PI/8-5.0*M_PI/180}" />
   </xacro:realsense>
 </robot>

File: kuka_control/models/ft_tool_real.xacro (robot description, xacro)
@@ -19,5 +19,5 @@
   <xacro:include filename="$(find kuka_control)/models/tool/tool.xacro"/>
   <xacro:tool parent="axia80_ft_measure" name="tool">
-    <origin xyz="0 0 ${0.013+0.027}" rpy="0 0 0"/>
+    <origin xyz="0 0 0.013" rpy="0 0 0"/>
   </xacro:tool>
   <!-- Include Realsense D435 camera frame -->

File: kuka_description/urdf/kr6r900sixx.urdf.xacro (robot description, xacro)
@@ -9,9 +9,9 @@
   <xacro:include filename="$(find kuka_description)/urdf/kr6r900sixx.xacro" />
   <!-- Include FT-sensor and tool -->
-  <!--<xacro:if value="$(arg gazebo)">
+  <xacro:if value="$(arg gazebo)">
   <xacro:include filename="$(find kuka_control)/models/ft_tool.xacro" />
   </xacro:if>
   <xacro:unless value="$(arg gazebo)">
   <xacro:include filename="$(find kuka_control)/models/ft_tool_real.xacro" />
-  </xacro:unless>-->
+  </xacro:unless>
 </robot>

Commit message: Car door model in Blender rotated and translated to origin. Urdf xacro file to spawn car door added.

File: kuka_control/models/camera/kinect_camera.urdf.xacro (robot description, xacro)
@@ -64,5 +64,5 @@
             <horizontal_fov>${60 * M_PI/180.0}</horizontal_fov>
             <image>
-              <format>R8G8B8</format>
+              <format>B8G8R8</format>
               <!--<width>640</width>
               <height>480</height>-->

File: kuka_control/models/car_door/car_door.urdf.xacro (robot description, xacro)
@@ -6,5 +6,5 @@
   <!-- Car door (Vito) -->
   <xacro:car_door name="door1" parent="cell_link">
-      <origin xyz="0.0 0.0 0.8" rpy="0 0 0" />
+      <origin xyz="0.0 0.0 0.15" rpy="0 0 0" />
   </xacro:car_door>
 </robot>

File: kuka_control/models/car_door/car_door_alone.xacro (robot description, xacro)
@@ -1,10 +1,9 @@
 <?xml version="1.0" ?>
-<robot name="car_door" xmlns:xacro="http://ros.org/wiki/xacro">
-  <xacro:macro name="car_door" params="name parent *origin">
-  <link name="${name}">
+<robot name="car_door_alone" xmlns:xacro="http://ros.org/wiki/xacro">
+  <link name="car_door">
       <inertial>
-          <mass value="10" />
+          <mass value="20" />
           <origin xyz="0 0 0" rpy="0 0 0" />
-          <inertia ixx="0.1" ixy="0" ixz="0" iyy="0.1" iyz="0" izz="0.1" />
+          <inertia ixx="1" ixy="0" ixz="0" iyy="1" iyz="0" izz="1" />
       </inertial>
       <visual name="visual">
@@ -26,9 +25,4 @@
       </collision>
   </link>
-  <joint name="${name}_joint" type="fixed">
-      <xacro:insert_block name="origin" />
-      <parent link="${parent}" />
-      <child link="${name}"/>
-  </joint>
 <!--
   <gazebo reference="${name}">
@@ -36,4 +30,3 @@
   </gazebo>
 -->
-  </xacro:macro>
 </robot>
