Commit message: Extrinsic calibrations for Kinect and Realsense. New functionalitites for kr6_hololens.py

File: kuka_control/models/camera/camera_manfrotto.urdf.xacro (robot description, xacro)
@@ -8,14 +8,17 @@
   <xacro:include filename="$(find kuka_control)/models/manfrotto/manfrotto.xacro" />
  <!--  Manfrotto 1 (mf1) -->
-  <xacro:manfrotto name="mf1" parent="cell_link" r1="${M_PI-24.0*M_PI/180.0}" r2="${-31.5*M_PI/180.0}" r3="${(27.1-13.5)*M_PI/180.0}">
-    <origin xyz="0.95 -1.01 1.015" rpy="0 ${90.0*M_PI/180.0} ${M_PI}" />
+  <!--<xacro:manfrotto name="mf1" parent="cell_link" r1="${M_PI-24.0*M_PI/180.0}" r2="${-31.5*M_PI/180.0}" r3="${(27.1-13.5)*M_PI/180.0}"> -->
+    <xacro:manfrotto name="mf1" parent="cell_cam" r1="${M_PI-24.0*M_PI/180.0}" r2="${-31.5*M_PI/180.0}" r3="${(27.1-13.5)*M_PI/180.0}">
+    <origin xyz="0.95 ${-1.01-0.02} ${1.015-0.02}" rpy="0 ${90.0*M_PI/180.0} ${M_PI}" />
   </xacro:manfrotto>
  <!--  Manfrotto 2 (mf2) 19.3-->
-  <xacro:manfrotto name="mf2" parent="cell_link" r1="${(9.5-0.2)*M_PI/180.0+M_PI}" r2="${34.5*M_PI/180.0}" r3="${(39.5-18.0)*M_PI/180.0}">
-    <origin xyz="-0.95 -1.01 1.015" rpy="0 ${90.0*M_PI/180.0} 0" />
+  <!--<xacro:manfrotto name="mf2" parent="cell_link" r1="${(9.5-0.2)*M_PI/180.0+M_PI}" r2="${(34.5-1.0)*M_PI/180.0}" r3="${(39.5-18.0)*M_PI/180.0}">-->
+    <xacro:manfrotto name="mf2" parent="cell_cam" r1="${(9.5-0.2)*M_PI/180.0+M_PI}" r2="${(34.5-1.0)*M_PI/180.0}" r3="${(39.5-18.0)*M_PI/180.0}">
+    <origin xyz="-0.95 ${-1.01+0.02-0.02} ${1.015-0.015-0.02}" rpy="0 ${90.0*M_PI/180.0} 0" />
   </xacro:manfrotto>
  <!--  Manfrotto 3 (mf3) -->
-  <xacro:manfrotto name="mf3" parent="cell_link" r1="${43.3*M_PI/180.0+45.0*M_PI/180.0}" r2="${0.0*M_PI/180.0}" r3="${(42.5+17.2)*M_PI/180.0}">
-    <origin xyz="-0.015 1.02 1.295" rpy="${180.0*M_PI/180.0} 0 ${180.0*M_PI/180.0}" />
+  <!--<xacro:manfrotto name="mf3" parent="cell_link" r1="${43.3*M_PI/180.0+45.0*M_PI/180.0}" r2="${0.0*M_PI/180.0}" r3="${(42.5+17.2)*M_PI/180.0}">-->
+    <xacro:manfrotto name="mf3" parent="cell_cam" r1="${43.3*M_PI/180.0+45.0*M_PI/180.0}" r2="${0.0*M_PI/180.0}" r3="${(42.5+17.2)*M_PI/180.0}">
+    <origin xyz="-0.015 ${1.02-0.02} ${1.295-0.02}" rpy="${180.0*M_PI/180.0} 0 ${180.0*M_PI/180.0}" />
   </xacro:manfrotto>
  <!--  Kinect sensors -->
@@ -24,5 +27,5 @@
   </xacro:kinect_camera>
   <xacro:kinect_camera name="camera2" parent="mf2_frame" gazebo="$(arg gazebo)">
-    <origin xyz="0.057 0 0.047" rpy="${0.3*M_PI/180.0} ${-0.1*M_PI/180.0} ${-0.1*M_PI/180.0}" />
+    <origin xyz="0.057 0 0.047" rpy="${(0.3-1.5)*M_PI/180.0} ${-0.1*M_PI/180.0} ${-0.1*M_PI/180.0}" />
   </xacro:kinect_camera>
   <xacro:kinect_camera name="camera3" parent="mf3_frame" gazebo="$(arg gazebo)">

File: kuka_control/models/cell/cell.xacro (robot description, xacro)
@@ -34,4 +34,11 @@
   </joint>
   <link name="cell_link"/>
+  <joint name="link_joint_cam" type="fixed">
+      <!--<origin xyz="0.005 -0.005 0.648" rpy="${1.05*3.1416/180} ${0.5*3.1416/180} ${0.0*3.1416/180}" />-->
+      <origin xyz="0.0 0.0 0.0" rpy="${1.05*3.1416/180} 0 0" />
+      <parent link="cell_link" />
+      <child link="cell_cam"/>
+  </joint>
+  <link name="cell_cam"/>
   <gazebo>
     <static>true</static>

File: kuka_control/models/ft_tool_real.xacro (robot description, xacro)
@@ -19,10 +19,11 @@
   <xacro:include filename="$(find kuka_control)/models/tool/tool.xacro"/>
   <xacro:tool parent="axia80_ft_measure" name="tool">
-    <origin xyz="0 0 0.013" rpy="0 0 0"/>
+    <origin xyz="0 0 ${0.013+0.027}" rpy="0 0 0"/>
   </xacro:tool>
   <!-- Include Realsense D435 camera frame -->
   <xacro:include filename="$(find kuka_control)/models/realsense/realsense_d435.xacro" />
   <xacro:realsense parent="brida_link" name="camera">
-      <origin xyz="0.0739 -0.0306 0.01" rpy="0 ${-M_PI/2} ${M_PI-M_PI/8}" />
+   <!--   <origin xyz="0.0739 -0.0306 0.01" rpy="0 ${-M_PI/2} ${M_PI-M_PI/8}" />-->
+	<origin xyz="0.13 0.05 0.025" rpy="${-2.0*M_PI/180} ${-M_PI/2+30.0*M_PI/180} ${M_PI+M_PI/8-5.0*M_PI/180}" />
   </xacro:realsense>
 </robot>

Commit message: Updates in the controllers and other stuff

File: kuka_control/models/camera/camera_manfrotto.urdf.xacro (robot description, xacro)
@@ -1,4 +1,4 @@
 <?xml version="1.0" encoding="utf-8"?>
-<robot name="cell" xmlns:xacro="http://ros.org/wiki/xacro">
+<robot name="camera_manfrotto" xmlns:xacro="http://ros.org/wiki/xacro">
   <xacro:arg name="gazebo" default="false"/>
   <!-- Depth cameras -->

File: kuka_control/models/camera/kinect_camera.urdf.xacro (robot description, xacro)
@@ -57,8 +57,8 @@
       </xacro:kinect_camera_model>
       <!-- Kinect camera for simulation -->
-      <xacro:if value="${gazebo=='true'}">
+      <xacro:if value="${gazebo}">
       <gazebo reference="${name}_depth_frame">
         <sensor type="depth" name="${name}">
-          <update_rate>30</update_rate>
+          <update_rate>10</update_rate>
           <camera>
             <horizontal_fov>${60 * M_PI/180.0}</horizontal_fov>
@@ -83,5 +83,6 @@
             <depthImageCameraInfoTopicName>${name}/depth/camera_info</depthImageCameraInfoTopicName>
             <pointCloudTopicName>${name}/depth/points</pointCloudTopicName>
-            <frameName>/cell/${name}_depth_optical_frame</frameName>
+            <!--<frameName>/cell/${name}_depth_optical_frame</frameName>-->
+            <frameName>${name}_depth_optical_frame</frameName>
           </plugin>
         </sensor>

File: kuka_control/models/ft_sensor/ft_sensor_ati.gazebo.xacro (robot description, xacro)
@@ -19,5 +19,5 @@
         <gaussianNoise>0.001</gaussianNoise>
       </plugin>
-	</gazebo>
+    </gazebo>
     </xacro:macro>
 </robot>

File: kuka_control/models/ft_sensor/ft_sensor_ati.urdf.xacro (robot description, xacro)
@@ -1,4 +1,4 @@
 <?xml version="1.0"?>
-<robot xmlns:xacro="http://ros.org/wiki/xacro" name="ft_sensor_ati">
+<robot name="ft_sensor_ati" xmlns:xacro="http://ros.org/wiki/xacro">
     <!-- Include all available models -->
     <xacro:include filename="$(find kuka_control)/models/ft_sensor/models.urdf.xacro"/>

File: kuka_control/models/tool/tool.xacro (robot description, xacro)
@@ -142,7 +142,7 @@
         <!--<turnGravityOff>false</turnGravityOff>
         <selfCollide>false</selfCollide>-->
-        <!--<mu1 value="0.1" />
-        <mu2 value="0.1" />-->
-        <mu value="0.1" />
+        <mu1 value="0.1" />
+        <mu2 value="0.1" />
+        <!--<mu value="0.1" />-->
         <kp  value="100000" />
         <kd  value="0.01" />

File: kuka_description/urdf/kr6r900sixx.gazebo.xacro (robot description, xacro)
@@ -41,7 +41,8 @@
     <joint name="joint_a1">
       <hardwareInterface>hardware_interface/EffortJointInterface</hardwareInterface>
+      <!--<hardwareInterface>hardware_interface/PositionJointInterface</hardwareInterface>-->
     </joint>
     <actuator name="motor1">
-      <hardwareInterface>hardware_interface/EffortJointInterface</hardwareInterface>
+      <!--<hardwareInterface>hardware_interface/EffortJointInterface</hardwareInterface>-->
       <mechanicalReduction>1</mechanicalReduction>
     </actuator>
@@ -51,7 +52,8 @@
     <joint name="joint_a2">
       <hardwareInterface>hardware_interface/EffortJointInterface</hardwareInterface>
+      <!--<hardwareInterface>hardware_interface/PositionJointInterface</hardwareInterface>-->
     </joint>
     <actuator name="motor2">
-      <hardwareInterface>hardware_interface/EffortJointInterface</hardwareInterface>
+      <!--<hardwareInterface>hardware_interface/EffortJointInterface</hardwareInterface>-->
       <mechanicalReduction>1</mechanicalReduction>
     </actuator>
@@ -61,7 +63,8 @@
     <joint name="joint_a3">
       <hardwareInterface>hardware_interface/EffortJointInterface</hardwareInterface>
+      <!--<hardwareInterface>hardware_interface/PositionJointInterface</hardwareInterface>-->
     </joint>
     <actuator name="motor3">
-      <hardwareInterface>hardware_interface/EffortJointInterface</hardwareInterface>
+      <!--<hardwareInterface>hardware_interface/EffortJointInterface</hardwareInterface>-->
       <mechanicalReduction>1</mechanicalReduction>
     </actuator>
@@ -71,7 +74,8 @@
     <joint name="joint_a4">
       <hardwareInterface>hardware_interface/EffortJointInterface</hardwareInterface>
+      <!--<hardwareInterface>hardware_interface/PositionJointInterface</hardwareInterface>-->
     </joint>
     <actuator name="motor4">
-      <hardwareInterface>hardware_interface/EffortJointInterface</hardwareInterface>
+      <!--<hardwareInterface>hardware_interface/EffortJointInterface</hardwareInterface>-->
       <mechanicalReduction>1</mechanicalReduction>
     </actuator>
@@ -81,7 +85,8 @@
     <joint name="joint_a5">
       <hardwareInterface>hardware_interface/EffortJointInterface</hardwareInterface>
+      <!--<hardwareInterface>hardware_interface/PositionJointInterface</hardwareInterface>-->
     </joint>
     <actuator name="motor5">
-      <hardwareInterface>hardware_interface/EffortJointInterface</hardwareInterface>
+      <!--<hardwareInterface>hardware_interface/EffortJointInterface</hardwareInterface>-->
       <mechanicalReduction>1</mechanicalReduction>
     </actuator>
@@ -91,9 +96,39 @@
     <joint name="joint_a6">
       <hardwareInterface>hardware_interface/EffortJointInterface</hardwareInterface>
+      <!--<hardwareInterface>hardware_interface/PositionJointInterface</hardwareInterface>-->
     </joint>
     <actuator name="motor6">
-      <hardwareInterface>hardware_interface/EffortJointInterface</hardwareInterface>
+      <!--<hardwareInterface>hardware_interface/EffortJointInterface</hardwareInterface>-->
       <mechanicalReduction>1</mechanicalReduction>
     </actuator>
   </transmission>
+  <!-- Gazebo-specific link properties -->
+  <!--<gazebo reference="base_link">
+    <material>Gazebo/Orange</material>
+    <turnGravityOff>true</turnGravityOff>
+  </gazebo>
+  <gazebo reference="link_1">
+    <material>Gazebo/Orange</material>
+    <turnGravityOff>true</turnGravityOff>
+  </gazebo>
+  <gazebo reference="link_2">
+    <material>Gazebo/Orange</material>
+    <turnGravityOff>true</turnGravityOff>
+  </gazebo>
+  <gazebo reference="link_3">
+    <material>Gazebo/Orange</material>
+    <turnGravityOff>true</turnGravityOff>
+  </gazebo>
+  <gazebo reference="link_4">
+    <material>Gazebo/Orange</material>
+    <turnGravityOff>true</turnGravityOff>
+  </gazebo>
+  <gazebo reference="link_5">
+    <material>Gazebo/Orange</material>
+    <turnGravityOff>true</turnGravityOff>
+  </gazebo>
+  <gazebo reference="link_6">
+    <material>Gazebo/Black</material>
+    <turnGravityOff>true</turnGravityOff>
+  </gazebo>-->
 </robot>

File: kuka_description/urdf/kr6r900sixx.urdf.xacro (robot description, xacro)
@@ -9,9 +9,9 @@
   <xacro:include filename="$(find kuka_description)/urdf/kr6r900sixx.xacro" />
   <!-- Include FT-sensor and tool -->
-  <xacro:if value="$(arg gazebo)">
+  <!--<xacro:if value="$(arg gazebo)">
   <xacro:include filename="$(find kuka_control)/models/ft_tool.xacro" />
   </xacro:if>
   <xacro:unless value="$(arg gazebo)">
   <xacro:include filename="$(find kuka_control)/models/ft_tool_real.xacro" />
-  </xacro:unless>
+  </xacro:unless>-->
 </robot>

File: kuka_description/urdf/kr6r900sixx_macro.xacro (robot description, xacro)
@@ -28,6 +28,6 @@
   <xacro:property name="diameter6" value="0.033" />
   <xacro:property name="max_effort" value="1200" />
-  <xacro:property name="damping" value="0.0"/>
-  <xacro:property name="friction" value="0.0"/>
+  <xacro:property name="damping" value="1.0"/>
+  <xacro:property name="friction" value="1.0"/>
   <xacro:macro name="kuka_kr6r900sixx" params="prefix">
     <link name="${prefix}base_link">

Commit message: Rviz configuration modified. Car door model added. Kinect reference frame updated to be compatible with real camera

File: kuka_control/models/camera/camera_manfrotto.urdf.xacro (robot description, xacro)
@@ -10,15 +10,15 @@
   <!--<xacro:manfrotto name="mf1" parent="cell_link" r1="${M_PI-24.0*M_PI/180.0}" r2="${-31.5*M_PI/180.0}" r3="${(27.1-13.5)*M_PI/180.0}"> -->
     <xacro:manfrotto name="mf1" parent="cell_cam" r1="${M_PI-24.0*M_PI/180.0}" r2="${-31.5*M_PI/180.0}" r3="${(27.1-13.5)*M_PI/180.0}">
-    <origin xyz="0.95 ${-1.01-0.02} ${1.015-0.02}" rpy="0 ${90.0*M_PI/180.0} ${M_PI}" />
+    <origin xyz="0.95 ${-1.01+0.02} ${1.015}" rpy="0 ${90.0*M_PI/180.0} ${M_PI}" />
   </xacro:manfrotto>
  <!--  Manfrotto 2 (mf2) 19.3-->
   <!--<xacro:manfrotto name="mf2" parent="cell_link" r1="${(9.5-0.2)*M_PI/180.0+M_PI}" r2="${(34.5-1.0)*M_PI/180.0}" r3="${(39.5-18.0)*M_PI/180.0}">-->
     <xacro:manfrotto name="mf2" parent="cell_cam" r1="${(9.5-0.2)*M_PI/180.0+M_PI}" r2="${(34.5-1.0)*M_PI/180.0}" r3="${(39.5-18.0)*M_PI/180.0}">
-    <origin xyz="-0.95 ${-1.01+0.02-0.02} ${1.015-0.015-0.02}" rpy="0 ${90.0*M_PI/180.0} 0" />
+    <origin xyz="-0.95 ${-1.01+0.02} ${1.015}" rpy="0 ${90.0*M_PI/180.0} 0" />
   </xacro:manfrotto>
  <!--  Manfrotto 3 (mf3) -->
   <!--<xacro:manfrotto name="mf3" parent="cell_link" r1="${43.3*M_PI/180.0+45.0*M_PI/180.0}" r2="${0.0*M_PI/180.0}" r3="${(42.5+17.2)*M_PI/180.0}">-->
     <xacro:manfrotto name="mf3" parent="cell_cam" r1="${43.3*M_PI/180.0+45.0*M_PI/180.0}" r2="${0.0*M_PI/180.0}" r3="${(42.5+17.2)*M_PI/180.0}">
-    <origin xyz="-0.015 ${1.02-0.02} ${1.295-0.02}" rpy="${180.0*M_PI/180.0} 0 ${180.0*M_PI/180.0}" />
+    <origin xyz="-0.015 ${1.02+0.02} ${1.295}" rpy="${180.0*M_PI/180.0} 0 ${180.0*M_PI/180.0}" />
   </xacro:manfrotto>
  <!--  Kinect sensors -->

File: kuka_control/models/camera/kinect_camera.urdf.xacro (robot description, xacro)
@@ -58,5 +58,5 @@
       <!-- Kinect camera for simulation -->
       <xacro:if value="${gazebo}">
-      <gazebo reference="${name}_depth_frame">
+      <gazebo reference="${name}_rgb_frame">
         <sensor type="depth" name="${name}">
           <update_rate>10</update_rate>
@@ -80,9 +80,9 @@
             <imageTopicName>${name}/rgb/image_raw</imageTopicName>
             <cameraInfoTopicName>${name}/rgb/camera_info</cameraInfoTopicName>
-            <depthImageTopicName>${name}/depth/image_raw</depthImageTopicName>
-            <depthImageCameraInfoTopicName>${name}/depth/camera_info</depthImageCameraInfoTopicName>
-            <pointCloudTopicName>${name}/depth/points</pointCloudTopicName>
+            <depthImageTopicName>${name}/depth_registered/image_raw</depthImageTopicName>
+            <depthImageCameraInfoTopicName>${name}/depth_registered/camera_info</depthImageCameraInfoTopicName>
+            <pointCloudTopicName>${name}/depth_registered/points</pointCloudTopicName>
             <!--<frameName>/cell/${name}_depth_optical_frame</frameName>-->
-            <frameName>${name}_depth_optical_frame</frameName>
+            <frameName>${name}_rgb_optical_frame</frameName>
           </plugin>
         </sensor>

File: kuka_control/models/car_door/car_door_alone.xacro (robot description, xacro)
@@ -10,5 +10,5 @@
         <geometry>
           <!--<mesh filename="package://kuka_control/models/car_door/meshes/car_door.dae"/>-->
-          <mesh filename="package://kuka_control/models/car_door/meshes/VITO_puerta_izq.dae"/>
+          <mesh filename="package://kuka_control/models/car_door/meshes/car_VITO.dae"/>
         </geometry>
         <!--
@@ -21,5 +21,5 @@
         <geometry>
           <!--<mesh filename="package://kuka_control/models/car_door/meshes/car_door.dae"/>-->
-          <mesh filename="package://kuka_control/models/car_door/meshes/VITO_puerta_izq.dae"/>
+          <mesh filename="package://kuka_control/models/car_door/meshes/car_VITO.dae"/>
         </geometry>
       </collision>
